File: stm32devBoardf405rg.kicad_sch (KiCad schematic)
At the start: 54 parts, among them J1 Screw_Terminal_01x02, J2 SWD, J3 Conn_01x04, J4 Conn_01x04, J5 USB_B_Micro, Q1 AO3401A, SW1 SW_SPDT, U1 STM32F405RGT6, U2 USBLC6-2SC6, Y1 16MZ

Commit message: finished with the placing of component
Connections:
- net +12V: now also Q1.3 (D); no longer F1.1
- net at D2.1 (K), Q1.2 (S): now also F1.1; no longer FB1.2
- net at F1.2: now also FB1.2; no longer Q1.3 (D)
Other:
- moved on the sheet: D2, F1, J1, Q1

Commit message: replaced swd footprint
Parts:
- J2: footprint Connector_PinSocket_1.27mm:PinSocket_2x05_P1.27mm_Vertical_SMD -> Connector_PinHeader_1.27mm:PinHeader_2x05_P1.27mm_Vertical_SMD
Changed lines of the file:
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@@
       (effects (font (size 1.27 1.27)))
     )
-    (property "Footprint" "Connector_PinSocket_1.27mm:PinSocket_2x05_P1.27mm_Vertical_SMD" (at 264.16 273.05 0)
+    (property "Footprint" "Connector_PinHeader_1.27mm:PinHeader_2x05_P1.27mm_Vertical_SMD" (at 264.16 273.05 0)
       (effects (font (size 1.27 1.27)) hide)
     )

Commit message: first STM32 board,final commit
Parts:
- C1, C2: LCSC Part# (none) -> C23630
- C10: LCSC Part# (none) -> C15195
- C11, C12: LCSC Part# (none) -> C1547
- C13, C14, C15, C16: LCSC Part# (none) -> C178330
- C3: LCSC Part# (none) -> C19666
- C4, C5, C6, C7, C8: LCSC Part# (none) -> C1525
- C9: LCSC Part# (none) -> C52923
- D1: LCSC Part# (none) -> C72041
- D2: LCSC Part# (none) -> C8598
- D3: LCSC Part# (none) -> C2286
- F1: LCSC Part# (none) -> C369159
- FB1: LCSC Part# (none) -> C1017
- L1: value 3u3 -> 39n; footprint Inductor_SMD:L_0805_2012Metric -> Capacitor_SMD:C_0402_1005Metric; LCSC Part# (none) -> C26443
- L2: value 3u3 -> 10uH; footprint Inductor_SMD:L_0805_2012Metric -> Inductor_SMD:L_Sunlord_MWSA0503S; LCSC Part# (none) -> C139506; now not fitted
- Q1: LCSC Part# (none) -> C15127
- R1: LCSC Part# (none) -> C25744
- R10, R11, R12, R13: LCSC Part# (none) -> C23345
- R14, R15: LCSC Part# (none) -> C25879
- R16, R8: LCSC Part# (none) -> C21190
- R2: LCSC Part# (none) -> C25118
- R3: LCSC Part# (none) -> C22843
- R4: LCSC Part# (none) -> C25803
- R5: LCSC Part# (none) -> C23231
- R6: LCSC Part# (none) -> C22984
- R7: LCSC Part# (none) -> C25804
- R9: LCSC Part# (none) -> C22966
- TPMP2359DJ1: renamed from TPMP1; LCSC Part# (none) -> C2959845
- U1: LCSC Part# (none) -> C15742
- U2: LCSC Part# (none) -> C7519
- Y1: LCSC Part# (none) -> C13738
